File: pcbs/STS1_EPS_BCC.kicad_sch (KiCad schematic)
At the start: 45 parts, among them Q1 SI7135DP-T1-GE3, U1 LTC4020EUHFPBF, U2 SI7272DP-T1-GE3, U3 SI7272DP-T1-GE3

Commit message: Worked on STS1_EPS_1 layout.
Connections:
- net CHARGING is gone; now on net BAT_CHARGING: R10.2
- net FAULT is gone; now on net BAT_FAULT: R11.2
- net +5V: now also D3.2 (A), D4.2 (A)
- net VOUT: no longer D3.2 (A), D4.2 (A)
Other:
- moved on the sheet: D4, R11
