File: pcbs/STS1_EPS_1_ORING.kicad_sch (KiCad schematic)
At the start: 4 parts, among them U27 LTC4451AV#TRMPBF, U28 LTC4451AV#TRMPBF

Commit message: Added testpoints to STS1_EPS_1.
Parts:
- added TP12, TP13: TestPoint, TestPoint:TestPoint_THTPad_D1.0mm_Drill0.5mm, symbol Connector:TestPoint
Connections:
- net GND: no longer U27.15 (STATUS), U28.15 (STATUS)
- new net: TP12.1, U27.15 (STATUS)
- new net: TP13.1, U28.15 (STATUS)
Changed lines of the file:
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@@
-    (pin "1")
-  )
-  (symbol (lib_id "power:GND") (at 92.71 52.07 90) (unit 1)
-    (in_bom yes) (on_board yes) (fields_autoplaced)
-    (property "Reference" "#PWR081" (id 0) (at 99.06 52.07 0)
-      (effects (font (size 1.27 1.27)) hide)
-    )
-    (property "Value" "GND" (id 1) (at 96.52 52.0699 90)
-      (effects (font (size 1.27 1.27)) (justify right))
-    )
-    (property "Footprint" "" (id 2) (at 92.71 52.07 0)
-      (effects (font (size 1.27 1.27)) hide)
-    )
-    (property "Datasheet" "" (id 3) (at 92.71 52.07 0)
-      (effects (font (size 1.27 1.27)) hide)
-    )
     (pin "1")
   )
@@
     )
     (property "Datasheet" "" (id 3) (at 93.98 123.19 0)
+      (effects (font (size 1.27 1.27)) hide)
+    )
+    (pin "1")
+  )
+  (symbol (lib_id "Connector:TestPoint") (at 92.71 52.07 270) (unit 1)
+    (in_bom yes) (on_board yes) (fields_autoplaced)
+    (property "Reference" "TP12" (id 0) (at 98.425 50.7999 90)
+      (effects (font (size 1.27 1.27)) (justify left))
+    )
+    (property "Value" "TestPoint" (id 1) (at 98.425 53.3399 90)
+      (effects (font (size 1.27 1.27)) (justify left))
+    )
+    (property "Footprint" "TestPoint:TestPoint_THTPad_D1.0mm_Drill0.5mm" (id 2) (at 92.71 57.15 0)
+      (effects (font (size 1.27 1.27)) hide)
+    )
+    (property "Datasheet" "~" (id 3) (at 92.71 57.15 0)
       (effects (font (size 1.27 1.27)) hide)
     )
@@
     (pin "1")
   )
-  (symbol (lib_id "power:GND") (at 93.98 118.11 90) (unit 1)
+  (symbol (lib_id "Connector:TestPoint") (at 93.98 118.11 270) (unit 1)
     (in_bom yes) (on_board yes) (fields_autoplaced)
-    (property "Reference" "#PWR084" (id 0) (at 100.33 118.11 0)
+    (property "Reference" "TP13" (id 0) (at 99.695 116.8399 90)
+      (effects (font (size 1.27 1.27)) (justify left))
+    )
+    (property "Value" "TestPoint" (id 1) (at 99.695 119.3799 90)
+      (effects (font (size 1.27 1.27)) (justify left))
+    )
+    (property "Footprint" "TestPoint:TestPoint_THTPad_D1.0mm_Drill0.5mm" (id 2) (at 93.98 123.19 0)
       (effects (font (size 1.27 1.27)) hide)
     )
-    (property "Value" "GND" (id 1) (at 97.79 118.1099 90)
-      (effects (font (size 1.27 1.27)) (justify right))
-    )
-    (property "Footprint" "" (id 2) (at 93.98 118.11 0)
+    (property "Datasheet" "~" (id 3) (at 93.98 123.19 0)
       (effects (font (size 1.27 1.27)) hide)
     )
-    (property "Datasheet" "" (id 3) (at 93.98 118.11 0)
-      (effects (font (size 1.27 1.27)) hide)
-    )

Commit message: Worked on STS1_EPS_1.
Parts:
- added C7: 100n, Capacitor_SMD:C_0805_2012Metric, symbol Device:C
Connections:
- net GND: now also C7.2
- net MPPT_BUS: now also C7.1
Changed lines of the file:
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@@
 (kicad_sch (version 20211123) (generator eeschema)
   (paper "A4")
+  (junction (at 49.53 113.03) (diameter 0) (color 0 0 0 0)
+  )
   (junction (at 49.53 46.99) (diameter 0) (color 0 0 0 0)
   )
@@
     (stroke (width 0) (type default) (color 0 0 0 0))
   )
+  (wire (pts (xy 49.53 113.03) (xy 49.53 114.935))
+    (stroke (width 0) (type default) (color 0 0 0 0))
+  )
   (wire (pts (xy 41.91 46.99) (xy 49.53 46.99))
     (stroke (width 0) (type default) (color 0 0 0 0))
@@
     (stroke (width 0) (type default) (color 0 0 0 0))
   )
+  (wire (pts (xy 49.53 122.555) (xy 49.53 125.73))
+    (stroke (width 0) (type default) (color 0 0 0 0))
+  )
   (wire (pts (xy 102.87 113.03) (xy 102.87 133.35))
     (stroke (width 0) (type default) (color 0 0 0 0))
   )
-  (wire (pts (xy 45.72 113.03) (xy 58.42 113.03))
+  (wire (pts (xy 45.72 113.03) (xy 49.53 113.03))
     (stroke (width 0) (type default) (color 0 0 0 0))
   )
@@
   )
   (wire (pts (xy 102.87 46.99) (xy 105.41 46.99))
+    (stroke (width 0) (type default) (color 0 0 0 0))
+  )
+  (wire (pts (xy 49.53 113.03) (xy 58.42 113.03))
     (stroke (width 0) (type default) (color 0 0 0 0))
   )
@@
   (hierarchical_label "VOUT" (shape input) (at 41.91 46.99 180)
     (effects (font (size 1.27 1.27)) (justify right))
+  )
+  (symbol (lib_id "Device:C") (at 49.53 118.745 0) (unit 1)
+    (in_bom yes) (on_board yes)
+    (property "Reference" "C7" (id 0) (at 50.8 114.935 0)
+      (effects (font (size 1.27 1.27)) (justify left))
+    )
+    (property "Value" "100n" (id 1) (at 50.8 122.555 0)
+      (effects (font (size 1.27 1.27)) (justify left))
+    )
+    (property "Footprint" "Capacitor_SMD:C_0805_2012Metric" (id 2) (at 50.4952 122.555 0)
+      (effects (font (size 1.27 1.27)) hide)
+    )
+    (property "Datasheet" "~" (id 3) (at 49.53 118.745 0)
+      (effects (font (size 1.27 1.27)) hide)
+    )
+    (pin "1")
+    (pin "2")
   )
   (symbol (lib_id "power:GND") (at 49.53 60.96 0) (unit 1)
@@
       (effects (font (size 1.27 1.27)) hide)
     )
+    (pin "1")
+  )
+  (symbol (lib_id "power:GND") (at 49.53 125.73 0) (unit 1)
+    (in_bom yes) (on_board yes) (fields_autoplaced)
+    (property "Reference" "#PWR072" (id 0) (at 49.53 132.08 0)
+      (effects (font (size 1.27 1.27)) hide)
+    )
+    (property "Value" "GND" (id 1) (at 52.07 126.9999 0)
+      (effects (font (size 1.27 1.27)) (justify left))
+    )
+    (property "Footprint" "" (id 2) (at 49.53 125.73 0)
+      (effects (font (size 1.27 1.27)) hide)
+    )
+    (property "Datasheet" "" (id 3) (at 49.53 125.73 0)
+      (effects (font (size 1.27 1.27)) hide)
+    )
