File: pcbs/STS1_EPS_2_CAP_BANK.kicad_sch (KiCad schematic)
At the start: 16 parts

Commit message: Worked on STS1_EPS_2.
Parts:
- renumbered C9 to C10, C10 to C11, C11 to C12, C12 to C13, C13 to C14, C14 to C15, C15 to C16, C16 to C17, C17 to C18, C18 to C19, C19 to C20, C20 to C21, C21 to C22, C6 to C7, C7 to C8, C8 to C9
Changed lines of the file:
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@@
   (symbol (lib_id "power:GND") (at 109.855 70.485 0) (unit 1)
     (in_bom yes) (on_board yes) (fields_autoplaced)
-    (property "Reference" "#PWR067" (id 0) (at 109.855 76.835 0)
+    (property "Reference" "#PWR083" (id 0) (at 109.855 76.835 0)
       (effects (font (size 1.27 1.27)) hide)
     )
@@
   (symbol (lib_id "power:GND") (at 65.405 70.485 0) (unit 1)
     (in_bom yes) (on_board yes) (fields_autoplaced)
-    (property "Reference" "#PWR060" (id 0) (at 65.405 76.835 0)
+    (property "Reference" "#PWR076" (id 0) (at 65.405 76.835 0)
       (effects (font (size 1.27 1.27)) hide)
     )
@@
   (symbol (lib_id "power:GND") (at 39.37 45.085 0) (unit 1)
     (in_bom yes) (on_board yes) (fields_autoplaced)
-    (property "Reference" "#PWR055" (id 0) (at 39.37 51.435 0)
+    (property "Reference" "#PWR071" (id 0) (at 39.37 51.435 0)
       (effects (font (size 1.27 1.27)) hide)
     )
@@
   (symbol (lib_id "Device:C") (at 92.075 66.675 0) (unit 1)
     (in_bom yes) (on_board yes) (fields_autoplaced)
-    (property "Reference" "C15" (id 0) (at 95.885 65.4049 0)
+    (property "Reference" "C16" (id 0) (at 95.885 65.4049 0)
       (effects (font (size 1.27 1.27)) (justify left))
     )
@@
   (symbol (lib_id "Device:C") (at 74.295 66.675 0) (unit 1)
     (in_bom yes) (on_board yes) (fields_autoplaced)
-    (property "Reference" "C12" (id 0) (at 78.105 65.4049 0)
+    (property "Reference" "C13" (id 0) (at 78.105 65.4049 0)
       (effects (font (size 1.27 1.27)) (justify left))
     )
@@
   (symbol (lib_id "power:GND") (at 56.515 70.485 0) (unit 1)
     (in_bom yes) (on_board yes) (fields_autoplaced)
-    (property "Reference" "#PWR058" (id 0) (at 56.515 76.835 0)
+    (property "Reference" "#PWR074" (id 0) (at 56.515 76.835 0)
       (effects (font (size 1.27 1.27)) hide)
     )
@@
   (symbol (lib_id "power:GND") (at 83.185 70.485 0) (unit 1)
     (in_bom yes) (on_board yes) (fields_autoplaced)
-    (property "Reference" "#PWR063" (id 0) (at 83.185 76.835 0)
+    (property "Reference" "#PWR079" (id 0) (at 83.185 76.835 0)
       (effects (font (size 1.27 1.27)) hide)
     )
@@
   (symbol (lib_id "power:GND") (at 113.665 45.085 0) (unit 1)
     (in_bom yes) (on_board yes) (fields_autoplaced)
-    (property "Reference" "#PWR068" (id 0) (at 113.665 51.435 0)
+    (property "Reference" "#PWR084" (id 0) (at 113.665 51.435 0)
       (effects (font (size 1.27 1.27)) hide)
     )
@@
   (symbol (lib_id "Device:C") (at 109.855 66.675 0) (unit 1)
     (in_bom yes) (on_board yes) (fields_autoplaced)
-    (property "Reference" "C18" (id 0) (at 113.665 65.4049 0)
+    (property "Reference" "C19" (id 0) (at 113.665 65.4049 0)
       (effects (font (size 1.27 1.27)) (justify left))
     )
@@
   (symbol (lib_id "power:GND") (at 120.015 70.485 0) (unit 1)
     (in_bom yes) (on_board yes) (fields_autoplaced)
-    (property "Reference" "#PWR069" (id 0) (at 120.015 76.835 0)
+    (property "Reference" "#PWR085" (id 0) (at 120.015 76.835 0)
       (effects (font (size 1.27 1.27)) hide)
     )
@@
   (symbol (lib_id "Device:C") (at 83.185 66.675 0) (unit 1)
     (in_bom yes) (on_board yes) (fields_autoplaced)
-    (property "Reference" "C14" (id 0) (at 86.995 65.4049 0)
+    (property "Reference" "C15" (id 0) (at 86.995 65.4049 0)
       (effects (font (size 1.27 1.27)) (justify left))
     )
@@
   (symbol (lib_id "power:GND") (at 92.075 70.485 0) (unit 1)
     (in_bom yes) (on_board yes) (fields_autoplaced)
-    (property "Reference" "#PWR064" (id 0) (at 92.075 76.835 0)
+    (property "Reference" "#PWR080" (id 0) (at 92.075 76.835 0)
       (effects (font (size 1.27 1.27)) hide)
     )
@@
   (symbol (lib_id "Device:C_Polarized") (at 58.42 38.735 0) (unit 1)
     (in_bom yes) (on_board yes) (fields_autoplaced)
-    (property "Reference" "C10" (id 0) (at 62.23 36.5759 0)
+    (property "Reference" "C11" (id 0) (at 62.23 36.5759 0)
       (effects (font (size 1.27 1.27)) (justify left))
     )
@@
   (symbol (lib_id "Device:C_Polarized") (at 39.37 38.735 0) (unit 1)
     (in_bom yes) (on_board yes) (fields_autoplaced)
-    (property "Reference" "C6" (id 0) (at 43.18 36.5759 0)
+    (property "Reference" "C7" (id 0) (at 43.18 36.5759 0)
       (effects (font (size 1.27 1.27)) (justify left))
     )
@@
   (symbol (lib_id "Device:C") (at 129.54 66.675 0) (unit 1)
     (in_bom yes) (on_board yes) (fields_autoplaced)
-    (property "Reference" "C21" (id 0) (at 133.35 65.4049 0)
+    (property "Reference" "C22" (id 0) (at 133.35 65.4049 0)
       (effects (font (size 1.27 1.27)) (justify left))
     )
@@
   (symbol (lib_id "power:GND") (at 129.54 70.485 0) (unit 1)
     (in_bom yes) (on_board yes) (fields_autoplaced)
-    (property "Reference" "#PWR070" (id 0) (at 129.54 76.835 0)
+    (property "Reference" "#PWR086" (id 0) (at 129.54 76.835 0)
       (effects (font (size 1.27 1.27)) hide)
     )
@@
   (symbol (lib_id "Device:C_Polarized") (at 95.885 38.735 0) (unit 1)
     (in_bom yes) (on_board yes) (fields_autoplaced)
-    (property "Reference" "C16" (id 0) (at 99.695 36.5759 0)
+    (property "Reference" "C17" (id 0) (at 99.695 36.5759 0)
       (effects (font (size 1.27 1.27)) (justify left))
     )
@@
   (symbol (lib_id "power:GND") (at 47.625 70.485 0) (unit 1)
     (in_bom yes) (on_board yes) (fields_autoplaced)
-    (property "Reference" "#PWR057" (id 0) (at 47.625 76.835 0)
+    (property "Reference" "#PWR073" (id 0) (at 47.625 76.835 0)
       (effects (font (size 1.27 1.27)) hide)
     )
@@
   (symbol (lib_id "Device:C") (at 39.37 66.675 0) (unit 1)
     (in_bom yes) (on_board yes) (fields_autoplaced)
-    (property "Reference" "C7" (id 0) (at 43.18 65.4049 0)
+    (property "Reference" "C8" (id 0) (at 43.18 65.4049 0)
       (effects (font (size 1.27 1.27)) (justify left))
     )
@@
   (symbol (lib_id "Device:C_Polarized") (at 77.47 38.735 0) (unit 1)
     (in_bom yes) (on_board yes) (fields_autoplaced)
-    (property "Reference" "C13" (id 0) (at 81.28 36.5759 0)
+    (property "Reference" "C14" (id 0) (at 81.28 36.5759 0)
       (effects (font (size 1.27 1.27)) (justify left))
     )
@@
   (symbol (lib_id "Device:C") (at 100.965 66.675 0) (unit 1)
     (in_bom yes) (on_board yes) (fields_autoplaced)
-    (property "Reference" "C17" (id 0) (at 104.775 65.4049 0)
+    (property "Reference" "C18" (id 0) (at 104.775 65.4049 0)
       (effects (font (size 1.27 1.27)) (justify left))
     )
@@
   (symbol (lib_id "power:GND") (at 58.42 45.085 0) (unit 1)
     (in_bom yes) (on_board yes) (fields_autoplaced)
-    (property "Reference" "#PWR059" (id 0) (at 58.42 51.435 0)
+    (property "Reference" "#PWR075" (id 0) (at 58.42 51.435 0)
       (effects (font (size 1.27 1.27)) hide)
     )
@@
   (symbol (lib_id "power:GND") (at 39.37 70.485 0) (unit 1)
     (in_bom yes) (on_board yes) (fields_autoplaced)
-    (property "Reference" "#PWR056" (id 0) (at 39.37 76.835 0)
+    (property "Reference" "#PWR072" (id 0) (at 39.37 76.835 0)
       (effects (font (size 1.27 1.27)) hide)
     )
@@
   (symbol (lib_id "Device:C_Polarized") (at 113.665 39.37 0) (unit 1)
     (in_bom yes) (on_board yes) (fields_autoplaced)
-    (property "Reference" "C19" (id 0) (at 117.475 37.2109 0)
+    (property "Reference" "C20" (id 0) (at 117.475 37.2109 0)
       (effects (font (size 1.27 1.27)) (justify left))
     )
@@
   (symbol (lib_id "Device:C") (at 120.015 66.675 0) (unit 1)
     (in_bom yes) (on_board yes) (fields_autoplaced)
-    (property "Reference" "C20" (id 0) (at 123.825 65.4049 0)
+    (property "Reference" "C21" (id 0) (at 123.825 65.4049 0)
       (effects (font (size 1.27 1.27)) (justify left))
     )
@@
   (symbol (lib_id "power:GND") (at 74.295 70.485 0) (unit 1)
     (in_bom yes) (on_board yes) (fields_autoplaced)
-    (property "Reference" "#PWR061" (id 0) (at 74.295 76.835 0)
+    (property "Reference" "#PWR077" (id 0) (at 74.295 76.835 0)
       (effects (font (size 1.27 1.27)) hide)
     )
@@
   (symbol (lib_id "Device:C") (at 56.515 66.675 0) (unit 1)
     (in_bom yes) (on_board yes) (fields_autoplaced)
-    (property "Reference" "C9" (id 0) (at 60.325 65.4049 0)
+    (property "Reference" "C10" (id 0) (at 60.325 65.4049 0)
       (effects (font (size 1.27 1.27)) (justify left))
     )
@@
   (symbol (lib_id "power:GND") (at 100.965 70.485 0) (unit 1)
     (in_bom yes) (on_board yes) (fields_autoplaced)
-    (property "Reference" "#PWR066" (id 0) (at 100.965 76.835 0)
+    (property "Reference" "#PWR082" (id 0) (at 100.965 76.835 0)
       (effects (font (size 1.27 1.27)) hide)
     )
@@
   (symbol (lib_id "Device:C") (at 65.405 66.675 0) (unit 1)
     (in_bom yes) (on_board yes) (fields_autoplaced)
-    (property "Reference" "C11" (id 0) (at 69.215 65.4049 0)
+    (property "Reference" "C12" (id 0) (at 69.215 65.4049 0)
       (effects (font (size 1.27 1.27)) (justify left))
     )
@@
   (symbol (lib_id "power:GND") (at 77.47 45.085 0) (unit 1)
     (in_bom yes) (on_board yes) (fields_autoplaced)
-    (property "Reference" "#PWR062" (id 0) (at 77.47 51.435 0)
+    (property "Reference" "#PWR078" (id 0) (at 77.47 51.435 0)
       (effects (font (size 1.27 1.27)) hide)
     )
@@
   (symbol (lib_id "Device:C") (at 47.625 66.675 0) (unit 1)
     (in_bom yes) (on_board yes) (fields_autoplaced)
-    (property "Reference" "C8" (id 0) (at 51.435 65.4049 0)
+    (property "Reference" "C9" (id 0) (at 51.435 65.4049 0)
       (effects (font (size 1.27 1.27)) (justify left))
     )
@@
   (symbol (lib_id "power:GND") (at 95.885 45.085 0) (unit 1)
     (in_bom yes) (on_board yes) (fields_autoplaced)
-    (property "Reference" "#PWR065" (id 0) (at 95.885 51.435 0)
-      (effects (font (size 1.27 1.27)) hide)
-    )
+    (property "Reference" "#PWR081" (id 0) (at 95.885 51.435 0)
+      (effects (font (size 1.27 1.27)) hide)
+    )
