File: pcbs/STS1_EPS_2_LOGIC_VOLTAGE.kicad_sch (KiCad schematic)
At the start: 7 parts, among them U11 LTC4451AV#TRMPBF, U12 LTC4451AV#TRMPBF

Commit message: Intermediate commit.
Connections:
- net GNDREF is gone; now on net GND: U11.14 (GND)
Other:
- moved on the sheet: C28, C6, TP15, TP19, U11, U12
