File: pcbs/STS1_EPS_SC_Connectors.kicad_sch (KiCad schematic)
At the start: 17 parts, among them J2 Panel Y-, J4 Panel Y+, J5 Panel Z-, J6 Panel Z+, J7 Panel X+, U25 TPS259472ARPW, U26 TPS259472ARPW, U29 TPS259472ARPW

Commit message: Fixed some warnings and errors.
Other:
- moved on the sheet: R54, R55
Changed lines of the file:
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@@
 	(wire
 		(pts
-			(xy 245.11 120.015) (xy 245.11 122.555)
+			(xy 245.11 120.65) (xy 245.11 123.19)
 		)
 		(stroke
@@
 	(wire
 		(pts
-			(xy 245.11 80.645) (xy 245.11 83.185)
+			(xy 245.11 81.28) (xy 245.11 83.82)
 		)
 		(stroke
@@
 	(wire
 		(pts
-			(xy 245.11 72.39) (xy 245.11 73.025)
+			(xy 245.11 72.39) (xy 245.11 73.66)
 		)
 		(stroke
@@
 	(wire
 		(pts
-			(xy 245.11 111.76) (xy 245.11 112.395)
+			(xy 245.11 111.76) (xy 245.11 113.03)
 		)
 		(stroke
@@
 	(text "Sets ~10 mA current limit."
 		(exclude_from_sim no)
-		(at 249.555 120.65 0)
+		(at 250.19 120.65 0)
 		(effects
 			(font
@@
 	(text "Overcurrent protection, reverse polarity protection"
 		(exclude_from_sim no)
-		(at 226.822 53.086 0)
+		(at 227.33 53.34 0)
 		(effects
 			(font
@@
 	(text "Sets ~4 A current limit."
 		(exclude_from_sim no)
-		(at 249.555 81.28 0)
+		(at 250.19 81.28 0)
 		(effects
 			(font
@@
 	(text "Ideal diode, that ensures\nthat the battery can not \nbe discharged via the UCI.\nAlso implements 13.8V \nover voltage lockout."
 		(exclude_from_sim no)
-		(at 212.344 90.932 0)
+		(at 212.09 91.44 0)
 		(effects
 			(font
@@
 	(text "Ideal diode, that protects\nthe COBC's UART\nAlso implements 5.7V \nover voltage lockout."
 		(exclude_from_sim no)
-		(at 213.106 129.032 0)
+		(at 213.36 129.54 0)
 		(effects
 			(font
@@
 			)
 		)
-		(property "Description" ""
+		(property "Description" "Power symbol creates a global label with name \"GND\" , ground"
 			(at 134.62 148.59 0)
 			(effects
@@
 			)
 		)
-		(property "Description" ""
+		(property "Description" "Power symbol creates a global label with name \"GND\" , ground"
 			(at 213.36 77.47 0)
 			(effects
@@
 	(symbol
 		(lib_id "Device:R")
-		(at 245.11 116.205 180)
+		(at 245.11 116.84 180)
 		(unit 1)
 		(exclude_from_sim no)
@@
 		(fields_autoplaced yes)
 		(property "Reference" "R55"
-			(at 247.015 114.9349 0)
+			(at 247.015 115.5699 0)
 			(effects
 				(font
@@
 		)
 		(property "Value" "332k"
-			(at 247.015 117.4749 0)
+			(at 247.015 118.1099 0)
 			(effects
 				(font
@@
 		)
 		(property "Footprint" "Resistor_SMD:R_0805_2012Metric"
-			(at 246.888 116.205 90)
+			(at 246.888 116.84 90)
 			(effects
 				(font
@@
 		)
 		(property "Datasheet" "~"
-			(at 245.11 116.205 0)
+			(at 245.11 116.84 0)
 			(effects
 				(font
@@
 		)
 		(property "Description" ""
-			(at 245.11 116.205 0)
+			(at 245.11 116.84 0)
 			(effects
 				(font
@@
 			)
 		)
-		(property "Description" ""
+		(property "Description" "Power symbol creates a global label with name \"GND\" , ground"
 			(at 213.36 148.59 0)
 			(effects
@@
 			)
 		)
-		(property "Description" ""
+		(property "Description" "Power symbol creates a global label with name \"GND\" , ground"
 			(at 64.77 40.64 0)
 			(effects
@@
 	(symbol
 		(lib_id "power:GND")
-		(at 245.11 83.185 0)
+		(at 245.11 83.82 0)
 		(unit 1)
 		(exclude_from_sim no)
@@
 		(fields_autoplaced yes)
 		(property "Reference" "#PWR079"
-			(at 245.11 89.535 0)
+			(at 245.11 90.17 0)
 			(effects
 				(font
@@
 		)
 		(property "Value" "GND"
-			(at 247.015 84.4549 0)
+			(at 245.11 88.265 0)
 			(effects
 				(font
 					(size 1.27 1.27)
 				)
-				(justify left)
 			)
 		)
 		(property "Footprint" ""
-			(at 245.11 83.185 0)
+			(at 245.11 83.82 0)
 			(effects
 				(font
@@
 		)
 		(property "Datasheet" ""
-			(at 245.11 83.185 0)
+			(at 245.11 83.82 0)
 			(effects
 				(font
@@
 			)
 		)
-		(property "Description" ""
-			(at 245.11 83.185 0)
+		(property "Description" "Power symbol creates a global label with name \"GND\" , ground"
+			(at 245.11 83.82 0)
 			(effects
 				(font
@@
 			)
 		)
-		(property "Description" ""
+		(property "Description" "Power symbol creates a global label with name \"GND\" , ground"
 			(at 64.77 87.63 0)
 			(effects
@@
 			)
 		)
-		(property "Description" ""
+		(property "Description" "Power symbol creates a global label with name \"GND\" , ground"
 			(at 213.36 151.13 0)
 			(effects
@@
 			)
 		)
-		(property "Description" ""
+		(property "Description" "Power symbol creates a global label with name \"GND\" , ground"
 			(at 139.7 95.25 0)
 			(effects
@@
 			)
 		)
-		(property "Description" ""
+		(property "Description" "Power symbol creates a global label with name \"GND\" , ground"
 			(at 213.36 74.93 0)
 			(effects
@@
 			)
 		)
-		(property "Description" ""
+		(property "Description" "Power symbol creates a global label with name \"GND\" , ground"
 			(at 139.7 71.12 0)
 			(effects
@@
 			)
 		)
-		(property "Description" ""
+		(property "Description" "Power symbol creates a global label with name \"GND\" , ground"
 			(at 64.77 63.5 0)
 			(effects
@@
 		)
 		(property "Value" "GND"
-			(at 247.015 157.4799 0)
+			(at 245.11 161.29 0)
 			(effects
 				(font
 					(size 1.27 1.27)
 				)
-				(justify left)
 			)
 		)
@@
 			)
 		)
-		(property "Description" ""
+		(property "Description" "Power symbol creates a global label with name \"GND\" , ground"
 			(at 245.11 156.21 0)
 			(effects
@@
 			)
 		)
-		(property "Description" ""
+		(property "Description" "Power symbol creates a global label with name \"GND\" , ground"
 			(at 234.95 148.59 0)
 			(effects
@@
 			)
 		)
-		(property "Description" ""
+		(property "Description" "Power symbol creates a global label with name \"GND\" , ground"
 			(at 139.7 120.65 0)
 			(effects
@@
 			)
 		)
-		(property "Description" ""
+		(property "Description" "Power symbol creates a global label with name \"GND\" , ground"
 			(at 234.95 74.93 0)
 			(effects
@@
 			)
 		)
-		(property "Description" ""
+		(property "Description" "Power symbol creates a global label with name \"GND\" , ground"
 			(at 134.62 74.93 0)
 			(effects
@@
 			)
 		)
-		(property "Description" ""
+		(property "Description" "Power symbol creates a global label with name \"GND\" , ground"
 			(at 134.62 124.46 0)
 			(effects
@@
 			)
 		)
-		(property "Description" ""
+		(property "Description" "Power symbol creates a global label with name \"GND\" , ground"
 			(at 139.7 118.11 0)
 			(effects
@@
 			)
 		)
-		(property "Description" ""
+		(property "Description" "Power symbol creates a global label with name \"GND\" , ground"
 			(at 129.54 118.11 0)
 			(effects
@@
 			)
 		)
-		(property "Description" ""
+		(property "Description" "Power symbol creates a global label with name \"GND\" , ground"
 			(at 64.77 149.86 0)
 			(effects
@@
 	(symbol
 		(lib_id "power:GND")
-		(at 245.11 122.555 0)
+		(at 245.11 123.19 0)
 		(unit 1)
 		(exclude_from_sim no)
@@
 		(fields_autoplaced yes)
 		(property "Reference" "#PWR095"
-			(at 245.11 128.905 0)
+			(at 245.11 129.54 0)
 			(effects
 				(font
@@
 		)
 		(property "Value" "GND"
-			(at 247.015 123.8249 0)
+			(at 245.11 127.635 0)
 			(effects
 				(font
 					(size 1.27 1.27)
 				)
-				(justify left)
 			)
 		)
 		(property "Footprint" ""
-			(at 245.11 122.555 0)
+			(at 245.11 123.19 0)
 			(effects
 				(font
@@
 		)
 		(property "Datasheet" ""
-			(at 245.11 122.555 0)
+			(at 245.11 123.19 0)
 			(effects
 				(font
@@
 			)
 		)
-		(property "Description" ""
-			(at 245.11 122.555 0)
+		(property "Description" "Power symbol creates a global label with name \"GND\" , ground"
+			(at 245.11 123.19 0)
 			(effects
 				(font
@@
 	(symbol
 		(lib_id "Device:R")
-		(at 245.11 76.835 180)
+		(at 245.11 77.47 180)
 		(unit 1)
 		(exclude_from_sim no)
@@
 		(fields_autoplaced yes)
 		(property "Reference" "R54"
-			(at 247.015 75.5649 0)
+			(at 247.015 76.1999 0)
 			(effects
 				(font
@@
 		)
 		(property "Value" "820"
-			(at 247.015 78.1049 0)
+			(at 247.015 78.7399 0)
 			(effects
 				(font
@@
 		)
 		(property "Footprint" "Resistor_SMD:R_0805_2012Metric"
-			(at 246.888 76.835 90)
+			(at 246.888 77.47 90)
 			(effects
 				(font
@@
 		)
 		(property "Datasheet" "~"
-			(at 245.11 76.835 0)
+			(at 245.11 77.47 0)
 			(effects
 				(font
@@
 		)
 		(property "Description" ""
-			(at 245.11 76.835 0)
+			(at 245.11 77.47 0)
 			(effects
 				(font
@@
 			)
 		)
-		(property "Description" ""
+		(property "Description" "Power symbol creates a global label with name \"GND\" , ground"
 			(at 139.7 144.78 0)
 			(effects
@@
 			)
 		)
-		(property "Description" ""
+		(property "Description" "Power symbol creates a global label with name \"GND\" , ground"
 			(at 134.62 99.06 0)
 			(effects
@@
 			)
 		)
-		(property "Description" ""
+		(property "Description" "Power symbol creates a global label with name \"GND\" , ground"
 			(at 234.95 114.3 0)
 			(effects
@@
 			)
 		)
-		(property "Description" ""
+		(property "Description" "Power symbol creates a global label with name \"GND\" , ground"
 			(at 134.62 175.26 0)
 			(effects
@@
 			)
 		)
-		(property "Description" ""
+		(property "Description" "Power symbol creates a global label with name \"GND\" , ground"
 			(at 191.77 72.39 0)
 			(effects
@@
 			)
 		)
-		(property "Description" ""
+		(property "Description" "Power symbol creates a global label with name \"GND\" , ground"
 			(at 64.77 111.76 0)
 			(effects
@@
 			)
 		)
-		(property "Description" ""
+		(property "Description" "Power symbol creates a global label with name \"GND\" , ground"
 			(at 213.36 114.3 0)
 			(effects
@@
 			)
 		)
-		(property "Description" ""
+		(property "Description" "Power symbol creates a global label with name \"GND\" , ground"
 			(at 129.54 120.65 0)
 			(effects
@@
 			)
 		)
-		(property "Description" ""
+		(property "Description" "Power symbol creates a global label with name \"GND\" , ground"
 			(at 213.36 116.84 0)
 			(effects
