File: pcbs/STS1_EPS_1_CurrentSources.kicad_sch (KiCad schematic)
At the start: 20 parts, among them U14 LM334M, U15 LM334M, U16 LM334M, U17 LM334M, U18 LM334M

Commit message: Added tolerances to some resistors that should be precise.
Parts:
- R26, R27, R28, R29, R30, R31, R32, R33, R34, R35: Tolerance (none) -> 1%
Changed lines of the file:
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@@
+	(wire
+		(pts
+			(xy 36.83 38.1) (xy 36.83 39.37)
+		)
+		(stroke
+			(width 0)
+			(type default)
+		)
+	)
 	(wire
 		(pts
@@
 		(pts
 			(xy 203.2 29.21) (xy 203.2 30.48)
-		)
-		(stroke
-			(width 0)
-			(type default)
-		)
-	)
-	(wire
-		(pts
-			(xy 36.83 38.1) (xy 36.83 39.37)
 		)
 		(stroke
@@
 		(on_board yes)
 		(dnp no)
-		(fields_autoplaced yes)
 		(property "Reference" "R28"
 			(at 77.47 33.0199 0)
@@
 				)
 				(hide yes)
+			)
+		)
+		(property "Tolerance" "1%"
+			(at 78.994 37.846 0)
+			(effects
+				(font
+					(size 1.27 1.27)
+				)
 			)
 		)
@@
 		(on_board yes)
 		(dnp no)
-		(fields_autoplaced yes)
 		(property "Reference" "R35"
 			(at 205.74 33.0199 0)
@@
 				)
 				(hide yes)
+			)
+		)
+		(property "Tolerance" "1%"
+			(at 207.264 37.592 0)
+			(effects
+				(font
+					(size 1.27 1.27)
+				)
 			)
 		)
@@
 		(on_board yes)
 		(dnp no)
-		(fields_autoplaced yes)
 		(property "Reference" "R32"
 			(at 157.48 33.0199 0)
@@
 				)
 				(hide yes)
+			)
+		)
+		(property "Tolerance" "1%"
+			(at 159.004 37.846 0)
+			(effects
+				(font
+					(size 1.27 1.27)
+				)
 			)
 		)
@@
 		(on_board yes)
 		(dnp no)
-		(fields_autoplaced yes)
 		(property "Reference" "R33"
 			(at 166.37 33.0199 0)
@@
 				)
 				(hide yes)
+			)
+		)
+		(property "Tolerance" "1%"
+			(at 167.894 37.592 0)
+			(effects
+				(font
+					(size 1.27 1.27)
+				)
 			)
 		)
@@
 		(on_board yes)
 		(dnp no)
-		(fields_autoplaced yes)
 		(property "Reference" "R34"
 			(at 196.85 33.0199 0)
@@
 				)
 				(hide yes)
+			)
+		)
+		(property "Tolerance" "1%"
+			(at 198.374 37.592 0)
+			(effects
+				(font
+					(size 1.27 1.27)
+				)
 			)
 		)
@@
 		(on_board yes)
 		(dnp no)
-		(fields_autoplaced yes)
 		(property "Reference" "R29"
 			(at 86.36 33.0199 0)
@@
 				)
 				(hide yes)
+			)
+		)
+		(property "Tolerance" "1%"
+			(at 87.884 37.846 0)
+			(effects
+				(font
+					(size 1.27 1.27)
+				)
 			)
 		)
@@
 		(on_board yes)
 		(dnp no)
-		(fields_autoplaced yes)
 		(property "Reference" "R31"
 			(at 125.73 33.0199 0)
@@
 				)
 				(hide yes)
+			)
+		)
+		(property "Tolerance" "1%"
+			(at 127.254 37.592 0)
+			(effects
+				(font
+					(size 1.27 1.27)
+				)
 			)
 		)
@@
 		(on_board yes)
 		(dnp no)
-		(fields_autoplaced yes)
 		(property "Reference" "R30"
 			(at 116.84 33.0199 0)
@@
 				)
 				(hide yes)
+			)
+		)
+		(property "Tolerance" "1%"
+			(at 118.364 37.592 0)
+			(effects
+				(font
+					(size 1.27 1.27)
+				)
 			)
 		)
@@
 		(on_board yes)
 		(dnp no)
-		(fields_autoplaced yes)
 		(property "Reference" "R27"
 			(at 48.26 33.0199 0)
@@
 				)
 				(hide yes)
+			)
+		)
+		(property "Tolerance" "1%"
+			(at 49.784 37.846 0)
+			(effects
+				(font
+					(size 1.27 1.27)
+				)
 			)
 		)
@@
 		(on_board yes)
 		(dnp no)
-		(fields_autoplaced yes)
 		(property "Reference" "R26"
 			(at 39.37 33.0199 0)
@@
 			)
 		)
+		(property "Tolerance" "1%"
+			(at 40.894 37.846 0)
+			(effects
+				(font
+					(size 1.27 1.27)
+				)
+			)
+		)

Commit message: Started adding part numbers to passive components.
Parts:
- D5, D6, D7, D8, D9: Part Nr. (none) -> TS4148 RYG
Changed lines of the file:
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@@
+			)
+		)
+		(property "Part Nr." "TS4148 RYG"
+			(at 185.42 45.72 0)
+			(effects
+				(font
+					(size 1.27 1.27)
+				)
+				(hide yes)
 			)
 		)
@@
 			)
 		)
+		(property "Part Nr." "TS4148 RYG"
+			(at 27.94 45.72 0)
+			(effects
+				(font
+					(size 1.27 1.27)
+				)
+				(hide yes)
+			)
+		)
 		(pin "1"
 		)
@@
 			)
 		)
+		(property "Part Nr." "TS4148 RYG"
+			(at 105.41 45.72 0)
+			(effects
+				(font
+					(size 1.27 1.27)
+				)
+				(hide yes)
+			)
+		)
 		(pin "1"
 		)
@@
 			)
 		)
+		(property "Part Nr." "TS4148 RYG"
+			(at 66.04 45.72 0)
+			(effects
+				(font
+					(size 1.27 1.27)
+				)
+				(hide yes)
+			)
+		)
 		(pin "1"
 		)
@@
 			(at 146.05 45.72 0)
 			(effects
+				(font
+					(size 1.27 1.27)
+				)
+				(hide yes)
+			)
+		)
+		(property "Part Nr." "TS4148 RYG"
+			(at 146.05 45.72 0)
+			(effects

Commit message: Added part numbers to components of STS1_EPS_1.
Parts:
- R26, R28, R30, R32, R34: Part Nr. (none) -> RT0805FRE07332RL
- R27, R29, R31, R33, R35: Part Nr. (none) -> RT0805FRE073K32L
Changed lines of the file:
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@@
+			)
+		)
+		(property "Part Nr." "RT0805FRE07332RL"
+			(at 74.93 34.29 0)
+			(effects
+				(font
+					(size 1.27 1.27)
+				)
+				(hide yes)
 			)
 		)
@@
 			)
 		)
+		(property "Part Nr." "RT0805FRE073K32L"
+			(at 203.2 34.29 0)
+			(effects
+				(font
+					(size 1.27 1.27)
+				)
+				(hide yes)
+			)
+		)
 		(pin "1"
 		)
@@
 			)
 		)
+		(property "Part Nr." "RT0805FRE07332RL"
+			(at 154.94 34.29 0)
+			(effects
+				(font
+					(size 1.27 1.27)
+				)
+				(hide yes)
+			)
+		)
 		(pin "1"
 		)
@@
 			)
 		)
+		(property "Part Nr." "RT0805FRE073K32L"
+			(at 163.83 34.29 0)
+			(effects
+				(font
+					(size 1.27 1.27)
+				)
+				(hide yes)
+			)
+		)
 		(pin "1"
 		)
@@
 			)
 		)
+		(property "Part Nr." "RT0805FRE07332RL"
+			(at 194.31 34.29 0)
+			(effects
+				(font
+					(size 1.27 1.27)
+				)
+				(hide yes)
+			)
+		)
 		(pin "1"
 		)
@@
 					(size 1.27 1.27)
 				)
+			)
+		)
+		(property "Part Nr." "RT0805FRE073K32L"
+			(at 83.82 34.29 0)
+			(effects
+				(font
+					(size 1.27 1.27)
+				)
+				(hide yes)
 			)
 		)
@@
 			)
 		)
+		(property "Part Nr." "RT0805FRE073K32L"
+			(at 123.19 34.29 0)
+			(effects
+				(font
+					(size 1.27 1.27)
+				)
+				(hide yes)
+			)
+		)
 		(pin "1"
 		)
@@
 			)
 		)
+		(property "Part Nr." "RT0805FRE07332RL"
+			(at 114.3 34.29 0)
+			(effects
+				(font
+					(size 1.27 1.27)
+				)
+				(hide yes)
+			)
+		)
 		(pin "1"
 		)
@@
 			)
 		)
+		(property "Part Nr." "RT0805FRE073K32L"
+			(at 45.72 34.29 0)
+			(effects
+				(font
+					(size 1.27 1.27)
+				)
+				(hide yes)
+			)
+		)
 		(pin "1"
 		)
@@
 			)
 		)
+		(property "Part Nr." "RT0805FRE07332RL"
+			(at 36.83 34.29 0)
+			(effects
+				(font
+					(size 1.27 1.27)
+				)
+				(hide yes)
+			)
+		)
