File: pcbs/STS1_EPS_1_MPPT_BUS_JUNCTION.kicad_sch (KiCad schematic)
At the start: 28 parts, among them Q2 SI7135DP-T1-GE3, Q3 SI7135DP-T1-GE3, U11 INA180A4, U13 TPS259472ARPW, U19 TPS259472ARPW, U20 TPS259472ARPW, U21 TPS259472ARPW, U22 TPS259472ARPW, U23 TPS259472ARPW, U24 TPS259472ARPW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

Commit message: Added tolerances to some resistors that should be precise.
Parts:
- R21, R22, R23, R39, R40, R41, R42, R46: value 6k8 -> 6k81; Tolerance (none) -> 1%
Changed lines of the file:
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@@
 	(text "Sets ~500 mA current limit."
 		(exclude_from_sim no)
-		(at 69.85 110.49 0)
+		(at 72.898 111.506 0)
 		(effects
 			(font
@@
 	(text "Sets ~500 mA current limit."
 		(exclude_from_sim no)
-		(at 69.85 35.56 0)
+		(at 71.882 36.576 0)
 		(effects
 			(font
@@
 	(text "Sets ~500 mA current limit."
 		(exclude_from_sim no)
-		(at 69.85 85.09 0)
+		(at 72.39 85.598 0)
 		(effects
 			(font
@@
 	(text "Sets ~500 mA current limit."
 		(exclude_from_sim no)
-		(at 69.85 162.56 0)
+		(at 72.644 163.83 0)
 		(effects
 			(font
@@
 	(text "Sets ~500 mA current limit."
 		(exclude_from_sim no)
-		(at 69.85 137.16 0)
+		(at 72.898 137.922 0)
 		(effects
 			(font
@@
 	(text "Sets ~500 mA current limit."
 		(exclude_from_sim no)
-		(at 69.85 58.42 0)
+		(at 72.39 58.928 0)
 		(effects
 			(font
@@
 	(text "Sets ~500 mA current limit."
 		(exclude_from_sim no)
-		(at 148.59 190.5 0)
+		(at 148.082 194.564 0)
 		(effects
 			(font
@@
 	(text "Sets ~500 mA current limit."
 		(exclude_from_sim no)
-		(at 69.85 189.23 0)
+		(at 72.644 190.246 0)
 		(effects
 			(font
@@
 		(on_board yes)
 		(dnp no)
-		(fields_autoplaced yes)
 		(property "Reference" "R46"
-			(at 66.675 30.4799 0)
+			(at 67.31 30.4799 0)
 			(effects
 				(font
@@
 			)
 		)
-		(property "Value" "6k8"
-			(at 66.675 33.0199 0)
+		(property "Value" "6k81"
+			(at 67.31 33.0199 0)
 			(effects
 				(font
@@
 			)
 		)
+		(property "Tolerance" "1%"
+			(at 68.58 35.306 0)
+			(effects
+				(font
+					(size 1.27 1.27)
+				)
+			)
+		)
 		(pin "1"
 		)
@@
 		(on_board yes)
 		(dnp no)
-		(fields_autoplaced yes)
 		(property "Reference" "R22"
 			(at 66.675 78.7399 0)
@@
 			)
 		)
-		(property "Value" "6k8"
+		(property "Value" "6k81"
 			(at 66.675 81.2799 0)
 			(effects
@@
 			)
 		)
+		(property "Tolerance" "1%"
+			(at 68.072 83.566 0)
+			(effects
+				(font
+					(size 1.27 1.27)
+				)
+			)
+		)
 		(pin "1"
 		)
@@
 		(on_board yes)
 		(dnp no)
-		(fields_autoplaced yes)
 		(property "Reference" "R39"
 			(at 66.675 130.8099 0)
@@
 			)
 		)
-		(property "Value" "6k8"
+		(property "Value" "6k81"
 			(at 66.675 133.3499 0)
 			(effects
@@
 			)
 		)
+		(property "Tolerance" "1%"
+			(at 68.072 135.89 0)
+			(effects
+				(font
+					(size 1.27 1.27)
+				)
+			)
+		)
 		(pin "1"
 		)
@@
 		(on_board yes)
 		(dnp no)
-		(fields_autoplaced yes)
 		(property "Reference" "R42"
 			(at 145.415 184.1499 0)
@@
 			)
 		)
-		(property "Value" "6k8"
+		(property "Value" "6k81"
 			(at 145.415 186.6899 0)
 			(effects
@@
 			)
 		)
+		(property "Tolerance" "1%"
+			(at 146.812 189.23 0)
+			(effects
+				(font
+					(size 1.27 1.27)
+				)
+			)
+		)
 		(pin "1"
 		)
@@
 		(on_board yes)
 		(dnp no)
-		(fields_autoplaced yes)
 		(property "Reference" "R41"
 			(at 66.675 184.1499 0)
@@
 			)
 		)
-		(property "Value" "6k8"
+		(property "Value" "6k81"
 			(at 66.675 186.6899 0)
 			(effects
@@
 			)
 		)
+		(property "Tolerance" "1%"
+			(at 68.072 188.976 0)
+			(effects
+				(font
+					(size 1.27 1.27)
+				)
+			)
+		)
 		(pin "1"
 		)
@@
 		(on_board yes)
 		(dnp no)
-		(fields_autoplaced yes)
 		(property "Reference" "R21"
 			(at 66.675 53.3399 0)
@@
 			)
 		)
-		(property "Value" "6k8"
+		(property "Value" "6k81"
 			(at 66.675 55.8799 0)
 			(effects
@@
 			)
 		)
+		(property "Tolerance" "1%"
+			(at 68.072 57.912 0)
+			(effects
+				(font
+					(size 1.27 1.27)
+				)
+			)
+		)
 		(pin "1"
 		)
@@
 		(on_board yes)
 		(dnp no)
-		(fields_autoplaced yes)
 		(property "Reference" "R40"
 			(at 66.675 157.4799 0)
@@
 			)
 		)
-		(property "Value" "6k8"
+		(property "Value" "6k81"
 			(at 66.675 160.0199 0)
 			(effects
@@
 			)
 		)
+		(property "Tolerance" "1%"
+			(at 68.072 162.306 0)
+			(effects
+				(font
+					(size 1.27 1.27)
+				)
+			)
+		)
 		(pin "1"
 		)
@@
 		(on_board yes)
 		(dnp no)
-		(fields_autoplaced yes)
 		(property "Reference" "R23"
 			(at 66.675 105.4099 0)
@@
 			)
 		)
-		(property "Value" "6k8"
+		(property "Value" "6k81"
 			(at 66.675 107.9499 0)
 			(effects
@@
 			)
 		)
+		(property "Tolerance" "1%"
+			(at 68.326 110.236 0)
+			(effects
+				(font
+					(size 1.27 1.27)
+				)
+			)
+		)

Commit message: Modified some resistor values slightly, so that they fall in common resistor series.
Parts:
- R44: Part Nr. (none) -> WFC0805R0100FE66; Tolerance (none) -> 1%
Changed lines of the file:
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@@
 		)
 		(property "Value" "10m"
-			(at 172.72 43.18 90)
+			(at 172.72 45.466 90)
 			(effects
 				(font
@@
 			(effects
 				(font
+					(size 1.27 1.27)
+				)
+				(hide yes)
+			)
+		)
+		(property "Tolerance" "1%"
+			(at 172.72 48.006 90)
+			(effects
+				(font
+					(size 1.27 1.27)
+				)
+			)
+		)
+		(property "Part Nr." "WFC0805R0100FE66"
+			(at 172.72 43.18 90)
+			(effects
+				(font

Commit message: Marked optional bypasses as "Do not place".
Parts:
- R37, R45: now not fitted
Changed lines of the file:
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@@
 		(in_bom yes)
 		(on_board yes)
-		(dnp no)
+		(dnp yes)
 		(property "Reference" "R45"
 			(at 210.82 20.32 90)
@@
 		(in_bom yes)
 		(on_board yes)
-		(dnp no)
+		(dnp yes)
 		(property "Reference" "R37"
 			(at 242.57 20.32 90)

Commit message: Changed net labels of the panel connectors, so they are consistent with the name of the respective connector.
Connections:
- net MPPT_X+_1_I: now also R41.2, U23.9 (ILM); no longer R46.2, U19.9 (ILM)
- net MPPT_X+_1_IN: now also U23.1 (EN/UVLO), U23.5 (IN); no longer U19.1 (EN/UVLO), U19.5 (IN)
- net MPPT_Y+_1_I: now also R22.2, U13.9 (ILM); no longer R39.2, U21.9 (ILM)
- net MPPT_Y+_1_IN: now also U13.1 (EN/UVLO), U13.5 (IN); no longer U21.1 (EN/UVLO), U21.5 (IN)
- net MPPT_Y+_2_I: now also R23.2, U20.9 (ILM); no longer R21.2, U4.9 (ILM)
- net MPPT_Y+_2_IN: now also U20.1 (EN/UVLO), U20.5 (IN); no longer U4.1 (EN/UVLO), U4.5 (IN)
- net MPPT_Y-_1_I: now also R39.2, U21.9 (ILM); no longer R22.2, U13.9 (ILM)
- net MPPT_Y-_1_IN: now also U21.1 (EN/UVLO), U21.5 (IN); no longer U13.1 (EN/UVLO), U13.5 (IN)
- net MPPT_Y-_2_I: now also R21.2, U4.9 (ILM); no longer R23.2, U20.9 (ILM)
- net MPPT_Y-_2_IN: now also U4.1 (EN/UVLO), U4.5 (IN); no longer U20.1 (EN/UVLO), U20.5 (IN)
- net MPPT_Z-_1_I: now also R46.2, U19.9 (ILM); no longer R41.2, U23.9 (ILM)
- net MPPT_Z-_1_IN: now also U19.1 (EN/UVLO), U19.5 (IN); no longer U23.1 (EN/UVLO), U23.5 (IN)
- net MPPT_X-_1_I renamed MPPT_Z+_1_I
- net MPPT_X-_1_IN renamed MPPT_Z+_1_IN
- net MPPT_Z-_2_I renamed MPPT_X+_2_I
- net MPPT_Z-_2_IN renamed MPPT_X+_2_IN

Commit message: Started adding part numbers to passive components.
Parts:
- Q2, Q3: Part Nr. (none) -> SI7135DP-T1-GE3
Changed lines of the file:
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@@
+			)
+		)
+		(property "Part Nr." "SI7135DP-T1-GE3"
+			(at 247.65 45.72 0)
+			(effects
+				(font
+					(size 1.27 1.27)
+				)
+				(hide yes)
 			)
 		)
@@
 				(hide yes)
 			)
+		)
+		(property "Part Nr." "SI7135DP-T1-GE3"
+			(at 215.9 45.72 0)
+			(effects
+				(font
+					(size 1.27 1.27)
+				)
+				(hide yes)
+			)

Commit message: Added part numbers to components of STS1_EPS_1.
Parts:
- R16, R17: Part Nr. (none) -> TNPW0805100KFEEA
- R21, R22, R23, R39, R40, R41, R42, R46: Part Nr. (none) -> MCU08050C6811FP500
Changed lines of the file:
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@@
 			)
 		)
+		(property "Part Nr." "MCU08050C6811FP500"
+			(at 64.77 31.75 0)
+			(effects
+				(font
+					(size 1.27 1.27)
+				)
+				(hide yes)
+			)
+		)
 		(pin "1"
 		)
@@
 			)
 		)
+		(property "Part Nr." "MCU08050C6811FP500"
+			(at 64.77 80.01 0)
+			(effects
+				(font
+					(size 1.27 1.27)
+				)
+				(hide yes)
+			)
+		)
 		(pin "1"
 		)
@@
 			)
 		)
+		(property "Part Nr." "MCU08050C6811FP500"
+			(at 64.77 132.08 0)
+			(effects
+				(font
+					(size 1.27 1.27)
+				)
+				(hide yes)
+			)
+		)
 		(pin "1"
 		)
@@
 			)
 		)
+		(property "Part Nr." "MCU08050C6811FP500"
+			(at 143.51 185.42 0)
+			(effects
+				(font
+					(size 1.27 1.27)
+				)
+				(hide yes)
+			)
+		)
 		(pin "1"
 		)
@@
 			)
 		)
+		(property "Part Nr." "MCU08050C6811FP500"
+			(at 64.77 185.42 0)
+			(effects
+				(font
+					(size 1.27 1.27)
+				)
+				(hide yes)
+			)
+		)
 		(pin "1"
 		)
@@
 			)
 		)
+		(property "Part Nr." "TNPW0805100KFEEA"
+			(at 229.87 48.26 0)
+			(effects
+				(font
+					(size 1.27 1.27)
+				)
+				(hide yes)
+			)
+		)
 		(pin "1"
 		)
@@
 			)
 		)
+		(property "Part Nr." "MCU08050C6811FP500"
+			(at 64.77 54.61 0)
+			(effects
+				(font
+					(size 1.27 1.27)
+				)
+				(hide yes)
+			)
+		)
 		(pin "1"
 		)
@@
 			)
 		)
+		(property "Part Nr." "MCU08050C6811FP500"
+			(at 64.77 158.75 0)
+			(effects
+				(font
+					(size 1.27 1.27)
+				)
+				(hide yes)
+			)
+		)
 		(pin "1"
 		)
@@
 			)
 		)
+		(property "Part Nr." "TNPW0805100KFEEA"
+			(at 198.12 48.26 0)
+			(effects
+				(font
+					(size 1.27 1.27)
+				)
+				(hide yes)
+			)
+		)
 		(pin "1"
 		)
@@
 			)
 		)
+		(property "Part Nr." "MCU08050C6811FP500"
+			(at 64.77 106.68 0)
+			(effects
+				(font
+					(size 1.27 1.27)
+				)
+				(hide yes)
+			)
+		)
